Commit message: WIP

File: src/openmower/description/lidar.xacro (robot description, xacro)
@@ -2,5 +2,5 @@
 <robot xmlns:xacro="http://www.ros.org/wiki/xacro" name="lidar">
     <joint name="lidar_joint" type="fixed">
-        <parent link="chassis"/>
+        <parent link="base_link"/>
         <child link="scan"/>
          <origin xyz="${robot['lidar']['sensor']['offset'][0]} ${robot['lidar']['sensor']['offset'][1]} ${robot['lidar']['sensor']['offset'][2]}" rpy="0 0 0"/>
@@ -9,5 +9,5 @@
     </link>
     <gazebo reference="scan">
-        <frame name="scan_frame" attached_to='chassis'>
+        <frame name="scan_frame" attached_to='base_link'>
             <pose relative_to='lidar_joint'>0 0 0 0 0 0</pose>
         </frame>
@@ -15,5 +15,5 @@
             <pose relative_to='scan_frame'>0 0 0 0 0 0</pose>
             <topic>scan</topic>
-            <update_rate>10</update_rate>
+            <update_rate>20</update_rate>
             <lidar>
                 <scan>
